Commit message: modified the urdf to change wrist roll to revolute instead of continuous

File: src/isaac_so_arm101/robots/pingti/urdf/PingTi_Arm_v3.urdf (robot description, URDF)
Before this commit: robot PingTi_Arm_v3, 16 links, 15 joints
Joints:
- joint elbow_pitch: axis -0.980528 -0.196381 0.0 -> -1 0 0; origin xyz=0.026719 -0.030548 0.0 rpy=0 0 0 -> xyz=0.026719 -0.030548 0.0 rpy=0 0 0.19635
- joint gripper_moving: axis -0.980528 -0.196381 -0.0 -> -1 0 0; origin xyz=0.019807 0.003967 0.0352 rpy=0 0 0 -> xyz=0.019807 0.003967 0.0352 rpy=0 0 0.19635
- joint shoulder_pitch: axis 0.980528 0.196381 -0.0 -> 1 0 0; origin xyz=0.019718 0.004408 0.03475 rpy=0 0 0 -> xyz=0.019718 0.004408 0.03475 rpy=0 0 0.19635
- joint wrist_pitch: axis -0.980528 -0.196381 -0.0 -> -1 0 0; origin xyz=-0.03236 -0.031417 -0.00045 rpy=0 0 0 -> xyz=-0.03236 -0.031417 -0.00045 rpy=0 0 0.19635
- joint wrist_roll: axis 0.196381 -0.980528 -0.0 -> 1 0 0; limit (none) -> lower=-3.14159 upper=3.14159 effort=100 velocity=100; origin xyz=0.009168 -0.037428 0.00045 rpy=0 0 0 -> xyz=0.009168 -0.037428 0.00045 rpy=0 0 -1.3744; type continuous -> revolute
