Commit message: modified the urdf wrist_roll joint type

File: src/isaac_so_arm101/robots/pingti/PingTi_Arm_5DOF_v4_copy.urdf (robot description, URDF)
Before this commit: robot PingTi_Arm_5DOF_v4_copy, 16 links, 15 joints
Joints:
- joint wrist_roll: limit (none) -> lower=-3.14159 upper=3.14159 effort=100 velocity=100; type continuous -> revolute

Commit message: updated the urdf file for the pingti arm

File: src/isaac_so_arm101/robots/pingti/PingTi_Arm_5DOF_v4_copy.urdf (robot description, URDF)
Before this commit: robot PingTi_Arm_5DOF_v4_copy, 16 links, 15 joints
Links:
- removed link STS3215_base_yaw_1
- removed link STS3215_elbow_pitch_1_1
- removed link STS3215_elbow_pitch_2_1
- removed link STS3215_gripper_1
- removed link STS3215_shoulder_pitch_1_1
- removed link STS3215_shoulder_pitch_2_1
- removed link STS3215_wrist_pitch_1
- removed link STS3215_wrist_roll_1
- removed link base_yaw_link_1
- removed link elbow_link_1
- removed link gripper_mount_1
- removed link moving_gripper_1
- removed link shoulder_link_1
- removed link wrist_link_1
- removed link wrist_mount_link_1
- added link base_yaw_link, mass 0.472148; collision mesh filename=package://pingti_arm_description/assets/base_yaw_link.stl; collision mesh filename=package://pingti_arm_description/assets/sts3215_shoulder_pi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
- added link moving_gripper, mass 0.0545806; collision mesh filename=package://pingti_arm_description/assets/moving_gripper.stl; visual mesh filename=package://pingti_arm_description/assets/moving_gripper.stl
- added link shoulder_link, mass 0.840414; collision mesh filename=package://pingti_arm_description/assets/shoulder_link.stl; collision mesh filename=package://pingti_arm_description/assets/sts3215_elbow_pitch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
- added link sts3215_gripper, mass 0.251542; collision mesh filename=package://pingti_arm_description/assets/gripper_mount.stl; collision mesh filename=package://pingti_arm_description/assets/sts3215_gripper.stl
- added link sts3215_wrist_roll, mass 0.176621; collision mesh filename=package://pingti_arm_description/assets/sts3215_wrist_roll.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; collision mesh filename=package://pingti_arm_description/assets/wrist_link.stl
- added link wrist_mount_link, mass 0.589063; collision mesh filename=package://pingti_arm_description/assets/elbow_link.stl; collision mesh filename=package://pingti_arm_description/assets/sts3215_wrist_pitch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
- link base_link: mass 1.1606702094747876 -> 0.42363; geometry collision mesh filename=package://pingti_arm_description/assets/base_link.stl; collision mesh filename=package://pingti_arm_description/assets/sts3215_base_yaw.stl
Joints:
- removed joint Rigid 24
- removed joint Rigid 25
- removed joint base_link_mount_connect
- removed joint base_yaw_link_servo_1_connect
- removed joint base_yaw_link_servo_2_connect
- removed joint elbow_wrist_servo_connect
- removed joint wrist_griper_mount_connect
- removed joint wrist_mount_connect
- removed joint wrist_wrist_roll_connect
- joint base_yaw: axis 0.0 0.0 -1.0 -> 0 0 1; child base_yaw_link_1 -> base_yaw_link; limit lower=-1.919862 upper=1.919862 effort=100 velocity=100 -> lower=-1.5708 upper=1.5708 effort=10 velocity=10; origin xyz=0.0 0.0102 -0.0183 rpy=0 0 0 -> xyz=-0.0109123 0.79568 0.127098 rpy=0 0 -1.5708; parent STS3215_base_yaw_1 -> base_link
- joint elbow_pitch: axis -1.0 0.0 -0.0 -> 0 0 1; child elbow_link_1 -> wrist_mount_link; limit lower=-1.570796 upper=1.919862 effort=100 velocity=100 -> lower=-1.44846 upper=1.69313 effort=10 velocity=10; origin xyz=0.0202 -0.0352 0.0 rpy=0 0 0 -> xyz=0.0317 0.23165 0.00195843 rpy=0 0 -0; parent STS3215_elbow_pitch_1_1 -> shoulder_link
- joint gripper_moving: axis 0.0 -0.0 1.0 -> 0 0 1; child moving_gripper_1 -> moving_gripper; limit lower=-0.20944 upper=1.570796 effort=100 velocity=100 -> lower=-0.0872665 upper=1.5708 effort=10 velocity=10; origin xyz=0.0352 0.0 -0.0202 rpy=0 0 0 -> xyz=0.013 0.0198025 -0.0234 rpy=1.5708 0 0; parent STS3215_gripper_1 -> sts3215_gripper
- joint shoulder_pitch: axis 1.0 -0.0 0.0 -> 0 0 1; child shoulder_link_1 -> shoulder_link; limit lower=-1.919862 upper=1.745329 effort=100 velocity=100 -> lower=-1.69313 upper=1.44846 effort=10 velocity=10; origin xyz=-0.0202 0.0 0.0352 rpy=0 0 0 -> xyz=0.03305 0.0391987 0.0928 rpy=1.5708 -0.122333 0; parent STS3215_shoulder_pitch_2_1 -> base_yaw_link
- joint wrist_pitch: axis -1.0 0.0 0.0 -> 0 0 1; child wrist_link_1 -> sts3215_wrist_roll; limit lower=-1.919862 upper=1.919862 effort=100 velocity=100 -> lower=-1.5708 upper=1.5708 effort=10 velocity=10; origin xyz=-0.0379 -0.02445 -0.00045 rpy=0 0 0 -> xyz=0.289534 -0.0335667 0.0154208 rpy=0 -0 -0.122333; parent STS3215_wrist_pitch_1 -> wrist_mount_link
- joint wrist_roll: axis 0.0 -1.0 -0.0 -> 0 0 1; child gripper_mount_1 -> sts3215_gripper; limit lower=-3.14159 upper=3.14159 effort=100 velocity=100 -> lower=-3.14159 upper=3.14159 effort=10 velocity=10; origin xyz=0.00164 -0.0385 0.00045 rpy=0 0 0 -> xyz=0.0624157 0 0.0185357 rpy=3.14159 1.5708 0; parent STS3215_wrist_roll_1 -> sts3215_wrist_roll

Commit message: re-exported the model from onshape after fixing the base_link coordinates

File: src/isaac_so_arm101/robots/pingti/PingTi_Arm_5DOF_v4_copy.urdf (robot description, URDF)
Before this commit: robot pingti_arm, 7 links, 6 joints
Joints:
- joint base_yaw: origin xyz=-0.0109123 0.79568 0.127098 rpy=0 0 -1.5708 -> xyz=-0 -0.00753894 0.0278 rpy=0 -0 -1.5708
- joint elbow_pitch: origin xyz=0.0317 0.23165 0.00195843 rpy=0 0 -0 -> xyz=0.0317 0.23165 0.00195843 rpy=0 -0 0
- joint shoulder_pitch: origin xyz=0.03305 0.0391987 0.0928 rpy=1.5708 -0.122333 0 -> xyz=0.03305 0.0391987 0.0928 rpy=1.5708 -0.122333 -0
